Commit message: Gazebo plugin finally working. Torque and velocity joint commands work.

File: bicycle_description/urdf/baseline_model.urdf.xacro (robot description, xacro)
@@ -191,13 +191,3 @@
     <dynamic damping="0" friction="0.002" />
   </joint>
-  <!--***********************************-->
-  <!--__________DUMMY LINK_______________-->
-  <!--***********************************-->
-  <link name="dummy_link">
-  </link>
-  <joint name="dummy" type="fixed">
-    <parent link="dummy_link"/>
-    <child link="back_frame"/>
-    <origin xyz="0 0 0" rpy="0 0 0"/>
-  </joint>
 </robot>

File: bicycle_description/urdf/baseline_model_rviz.urdf.xacro (robot description, xacro)
@@ -149,6 +149,6 @@
   <!--_________FRONT WHEEL LINK___________-->
   <!--***********************************-->
-   <!--link name="front_wheel">
-    <visual>
+   <link name="front_wheel">
+    <!--visual>
       <origin rpy="0 0 0" xyz="0 0 0"/>
       <geometry>
